Commit message: fine adjustment

File: darwin_description/urdf/hand.urdf.xacro (robot description, xacro)
@@ -1,20 +1,32 @@
 <?xml version="1.0"?>
 <robot xmlns:sensor="http://playerstage.sourceforge.net/gazebo/xmlschema/#sensor"
-    xmlns:controller="http://playerstage.sourceforge.net/gazebo/xmlschema/#controller"
-    xmlns:interface="http://playerstage.sourceforge.net/gazebo/xmlschema/#interface"
-    xmlns:xacro="http://www.ros.org/wiki/xacro">
-    <xacro:macro name="darwin_hand" params="side parent reflect">
-        <xacro:darwin_spo5 name="${side}_hand_wrist1" parent="${parent}" xyz="0 0.0015 0" rpy="0 0 0" />
-        <xacro:darwin_spo5 name="${side}_hand_wrist2" parent="${side}_hand_wrist1_link" xyz="0 0.003 0" rpy="0 0 0" />
-        <xacro:darwin_spd3b5 name="${side}_hand_base" parent="${side}_hand_wrist2_link" xyz="0 0.0045 0" rpy="0 ${M_PI/2} 0" />
-        <xacro:darwin_spl2b2 name="${side}_hand_thumb" parent="${side}_hand_base_link" xyz="0.018 0.0015 ${reflect*-0.009}" rpy="${M_PI/2} ${M_PI} 0" />
-        <xacro:darwin_spl2b2 name="${side}_hand_palm_anchor1" parent="${side}_hand_base_link" xyz="0.003 0.0015 ${reflect*0.012}" rpy="${M_PI/2} ${reflect*M_PI/2} 0" />
-        <xacro:darwin_spl2b2 name="${side}_hand_palm_anchor2" parent="${side}_hand_base_link" xyz="-0.009 0.0015 ${reflect*0.012}" rpy="${M_PI/2} ${reflect*M_PI/2} 0" />
-        <xacro:darwin_spd3b5 name="${side}_hand_palm" parent="${side}_hand_base_link" xyz="0 0.006 0" rpy="0 0 0" />
-        <xacro:darwin_spd4b5 name="${side}_hand_back" parent="${side}_hand_palm_anchor2_link" xyz="-0.0015 ${reflect*0.006} -0.015" rpy="0 ${M_PI/2} ${M_PI/2}" />
-        <xacro:darwin_spl2b2 name="${side}_hand_fingers_ext1" parent="${side}_hand_back_link" xyz="0.021 -0.0015 -0.006" rpy="${-M_PI/2} 0 ${-M_PI/2}" />
-        <xacro:darwin_spl2b2 name="${side}_hand_fingers_ext2" parent="${side}_hand_back_link" xyz="0.021 -0.0015 0.006" rpy="${-M_PI/2} 0 ${-M_PI/2}" />
-        <xacro:darwin_spl2b2 name="${side}_hand_fingers_int1" parent="${side}_hand_fingers_ext1_link" xyz="0.003 0 -0.003" rpy="${M_PI} ${M_PI/2} 0" />
-        <xacro:darwin_spl2b2 name="${side}_hand_fingers_int2" parent="${side}_hand_fingers_ext2_link" xyz="0.003 0 -0.003" rpy="${M_PI} ${M_PI/2} 0" />
-    </xacro:macro>
+       xmlns:controller="http://playerstage.sourceforge.net/gazebo/xmlschema/#controller"
+       xmlns:interface="http://playerstage.sourceforge.net/gazebo/xmlschema/#interface"
+       xmlns:xacro="http://www.ros.org/wiki/xacro">
+  <xacro:macro name="darwin_hand" params="side parent reflect">
+    <xacro:darwin_spo5 name="${side}_hand_wrist1" parent="${parent}"
+        xyz="0 0.0015 0" rpy="0 0 0" />
+    <xacro:darwin_spo5 name="${side}_hand_wrist2" parent="${side}_hand_wrist1_link"
+        xyz="0 0.003 0" rpy="0 0 0" />
+    <xacro:darwin_spd3b5 name="${side}_hand_base" parent="${side}_hand_wrist2_link"
+        xyz="0 0.0045 0" rpy="0 ${M_PI/2} 0" />
+    <xacro:darwin_spl2b2 name="${side}_hand_thumb" parent="${side}_hand_base_link"
+        xyz="0.018 0.0015 ${reflect*-0.009}" rpy="${M_PI/2} ${M_PI} 0" />
+    <xacro:darwin_spl2b2 name="${side}_hand_palm_anchor1" parent="${side}_hand_base_link"
+        xyz="0.003 0.0015 ${reflect*0.012}" rpy="${M_PI/2} ${reflect*M_PI/2} 0" />
+    <xacro:darwin_spl2b2 name="${side}_hand_palm_anchor2" parent="${side}_hand_base_link"
+        xyz="-0.009 0.0015 ${reflect*0.012}" rpy="${M_PI/2} ${reflect*M_PI/2} 0" />
+    <xacro:darwin_spd3b5 name="${side}_hand_palm" parent="${side}_hand_base_link"
+        xyz="0 0.006 0" rpy="0 0 0" />
+    <xacro:darwin_spd4b5 name="${side}_hand_back" parent="${side}_hand_palm_anchor2_link"
+        xyz="-0.0015 ${reflect*0.006} -0.015" rpy="0 ${M_PI/2} ${M_PI/2}" />
+    <xacro:darwin_spl2b2 name="${side}_hand_fingers_ext1" parent="${side}_hand_back_link"
+        xyz="0.021 -0.0015 -0.006" rpy="${-M_PI/2} 0 ${-M_PI/2}" />
+    <xacro:darwin_spl2b2 name="${side}_hand_fingers_ext2" parent="${side}_hand_back_link"
+        xyz="0.021 -0.0015 0.006" rpy="${-M_PI/2} 0 ${-M_PI/2}" />
+    <xacro:darwin_spl2b2 name="${side}_hand_fingers_int1" parent="${side}_hand_fingers_ext1_link"
+        xyz="0.003 0 -0.003" rpy="${M_PI} ${M_PI/2} 0" />
+    <xacro:darwin_spl2b2 name="${side}_hand_fingers_int2" parent="${side}_hand_fingers_ext2_link"
+        xyz="0.003 0 -0.003" rpy="${M_PI} ${M_PI/2} 0" />
+  </xacro:macro>
 </robot>
