Commit message: Head and arms ready

File: darwin_control/urdf/darwin_ctrl.urdf.xacro (robot description, xacro)
@@ -20,4 +20,72 @@
         </joint>
         <!-- LEFT ARM -->
+        <joint name="l_shoulder_joint">
+            <command_interface name="position">
+                <param name="min">1.047</param>
+                <param name="max">4.132</param>
+            </command_interface>
+            <state_interface name="position">
+                <param name="initial_value">0.0</param>
+            </state_interface>
+            <state_interface name="velocity"/>
+            <state_interface name="effort"/>
+        </joint>
+        <joint name="l_biceps_joint">
+            <command_interface name="position">
+                <param name="min">3.841</param>
+                <param name="max">4.104</param>
+            </command_interface>
+            <state_interface name="position">
+                <param name="initial_value">0.0</param>
+            </state_interface>
+            <state_interface name="velocity"/>
+            <state_interface name="effort"/>
+        </joint>
+        <joint name="l_elbow_joint">
+            <command_interface name="position">
+                <param name="min">1.302</param>
+                <param name="max">4.274</param>
+            </command_interface>
+            <state_interface name="position">
+                <param name="initial_value">0.0</param>
+            </state_interface>
+            <state_interface name="velocity"/>
+            <state_interface name="effort"/>
+        </joint>
+        <!-- RIGHT ARM -->
+        <joint name="r_shoulder_joint">
+            <command_interface name="position">
+                <param name="min">1.189</param>
+                <param name="max">4.161</param>
+            </command_interface>
+            <state_interface name="position">
+                <param name="initial_value">0.0</param>
+            </state_interface>
+            <state_interface name="velocity"/>
+            <state_interface name="effort"/>
+        </joint>
+        <joint name="r_biceps_joint">
+            <command_interface name="position">
+                <param name="min">0.906</param>
+                <param name="max">1.175</param>
+            </command_interface>
+            <state_interface name="position">
+                <param name="initial_value">0.0</param>
+            </state_interface>
+            <state_interface name="velocity"/>
+            <state_interface name="effort"/>
+        </joint>
+        <joint name="r_elbow_joint">
+            <command_interface name="position">
+                <param name="min">0.594</param>
+                <param name="max">3.764</param>
+            </command_interface>
+            <state_interface name="position">
+                <param name="initial_value">0.0</param>
+            </state_interface>
+            <state_interface name="velocity"/>
+            <state_interface name="effort"/>
+        </joint>
+        <!-- LEFT LEG -->
     </ros2_control>
 </robot>

Commit message: darwin_ctrl urdf xacro file completed

File: darwin_control/urdf/darwin_ctrl.urdf.xacro (robot description, xacro)
@@ -14,5 +14,5 @@
             </command_interface>
             <state_interface name="position">
-                <param name="initial_value">0.0</param>
+                <param name="initial_value">0.1</param>
             </state_interface>
             <state_interface name="velocity"/>
@@ -26,5 +26,5 @@
             </command_interface>
             <state_interface name="position">
-                <param name="initial_value">0.0</param>
+                <param name="initial_value">1.1</param>
             </state_interface>
             <state_interface name="velocity"/>
@@ -37,5 +37,5 @@
             </command_interface>
             <state_interface name="position">
-                <param name="initial_value">0.0</param>
+                <param name="initial_value">3.9</param>
             </state_interface>
             <state_interface name="velocity"/>
@@ -48,5 +48,5 @@
             </command_interface>
             <state_interface name="position">
-                <param name="initial_value">0.0</param>
+                <param name="initial_value">1.4</param>
             </state_interface>
             <state_interface name="velocity"/>
@@ -60,5 +60,5 @@
             </command_interface>
             <state_interface name="position">
-                <param name="initial_value">0.0</param>
+                <param name="initial_value">1.2</param>
             </state_interface>
             <state_interface name="velocity"/>
@@ -71,5 +71,5 @@
             </command_interface>
             <state_interface name="position">
-                <param name="initial_value">0.0</param>
+                <param name="initial_value">1.0</param>
             </state_interface>
             <state_interface name="velocity"/>
@@ -82,5 +82,5 @@
             </command_interface>
             <state_interface name="position">
-                <param name="initial_value">0.0</param>
+                <param name="initial_value">0.7</param>
             </state_interface>
             <state_interface name="velocity"/>
@@ -88,4 +88,115 @@
         </joint>
         <!-- LEFT LEG -->
+        <joint name="l_hip_joint">
+            <command_interface name="position">
+                <param name="min">0.000</param>
+                <param name="max">0.113</param>
+            </command_interface>
+            <state_interface name="position">
+                <param name="initial_value">0.0</param>
+            </state_interface>
+            <state_interface name="velocity"/>
+            <state_interface name="effort"/>
+        </joint>
+        <joint name="l_thigh_joint">
+            <command_interface name="position">
+                <param name="min">0.000</param>
+                <param name="max">0.200</param>
+            </command_interface>
+            <state_interface name="position">
+                <param name="initial_value">0.0</param>
+            </state_interface>
+            <state_interface name="velocity"/>
+            <state_interface name="effort"/>
+        </joint>
+        <joint name="l_knee_joint">
+            <command_interface name="position">
+                <param name="min">0.991</param>
+                <param name="max">3.142</param>
+            </command_interface>
+            <state_interface name="position">
+                <param name="initial_value">1.0</param>
+            </state_interface>
+            <state_interface name="velocity"/>
+            <state_interface name="effort"/>
+        </joint>
+        <joint name="l_ankle_joint">
+            <command_interface name="position">
+                <param name="min">0.991</param>
+                <param name="max">3.142</param>
+            </command_interface>
+            <state_interface name="position">
+                <param name="initial_value">1.0</param>
+            </state_interface>
+            <state_interface name="velocity"/>
+            <state_interface name="effort"/>
+        </joint>
+        <joint name="l_foot_joint">
+            <command_interface name="position">
+                <param name="min">3.764</param>
+                <param name="max">5.236</param>
+            </command_interface>
+            <state_interface name="position">
+                <param name="initial_value">3.9</param>
+            </state_interface>
+            <state_interface name="velocity"/>
+            <state_interface name="effort"/>
+        </joint>
+        <!-- RIGHT LEG -->
+        <joint name="r_hip_joint">
+            <command_interface name="position">
+                <param name="min">5.000</param>
+                <param name="max">5.236</param>
+            </command_interface>
+            <state_interface name="position">
+                <param name="initial_value">5.1</param>
+            </state_interface>
+            <state_interface name="velocity"/>
+            <state_interface name="effort"/>
+        </joint>
+        <joint name="r_thigh_joint">
+            <command_interface name="position">
+                <param name="min">0.000</param>
+                <param name="max">1.019</param>
+            </command_interface>
+            <state_interface name="position">
+                <param name="initial_value">0.0</param>
+            </state_interface>
+            <state_interface name="velocity"/>
+            <state_interface name="effort"/>
+        </joint>
+        <joint name="r_knee_joint">
+            <command_interface name="position">
+                <param name="min">0.793</param>
+                <param name="max">2.434</param>
+            </command_interface>
+            <state_interface name="position">
+                <param name="initial_value">0.9</param>
+            </state_interface>
+            <state_interface name="velocity"/>
+            <state_interface name="effort"/>
+        </joint>
+        <joint name="r_ankle_joint">
+            <command_interface name="position">
+                <param name="min">0.000</param>
+                <param name="max">1.302</param>
+            </command_interface>
+            <state_interface name="position">
+                <param name="initial_value">0.9</param>
+            </state_interface>
+            <state_interface name="velocity"/>
+            <state_interface name="effort"/>
+        </joint>
+        <joint name="r_foot_joint">
+            <command_interface name="position">
+                <param name="min">0.000</param>
+                <param name="max">1.132</param>
+            </command_interface>
+            <state_interface name="position">
+                <param name="initial_value">0.0</param>
+            </state_interface>
+            <state_interface name="velocity"/>
+            <state_interface name="effort"/>
+        </joint>
     </ros2_control>
 </robot>
